File: P.01_ISO/P.01_ISO.kicad_pcb (KiCad board)
At the start: 2 copper layers, 358.1 x 126.4 mm, 56 parts

Commit message: added plate files for all strata variants
Other:
- net class Default removed
