File: P.02_ANSI/P.02_ANSI.kicad_pcb (KiCad board)
At the start: 2 copper layers, 324.8 x 106.2 mm, 0 parts

Commit message: added plate files for all strata variants
Other:
- outline, holes or cut-outs redrawn
- net class Default removed
